File: talk2hand.sch (KiCad schematic (older format))
At the start: 4 parts, among them J1 USB_A, J2 USB_A

Commit message: PCB updates
Parts:
- D1: footprint LED_SMD:LED_0603_1608Metric_Pad1.05x0.95mm_HandSolder -> BBS Components:LED_0603_HandSoldering
- J1: footprint Connector_USB:USB_A_Stewart_SS-52100-001_Horizontal -> BBS Components:USB_B_Male_Molex_0480370001
- J2: footprint Connector_USB:USB_A_Stewart_SS-52100-001_Horizontal -> BBS Components:USB_A_Female_Molex_0676432910
- R1: footprint Resistor_SMD:R_0603_1608Metric_Pad1.05x0.95mm_HandSolder -> BBS Components:R_0603_HandSoldering_NoSilk
Changed lines of the file:
@@
 EESchema Schematic File Version 4
-EELAYER 30 0
+LIBS:talk2hand-cache
+EELAYER 29 0
 EELAYER END
 $Descr A4 11693 8268
@@
 F 0 "J1" H 1707 2217 50  0000 C CNN
 F 1 "USB_A" H 1707 2126 50  0000 C CNN
-F 2 "Connector_USB:USB_A_Stewart_SS-52100-001_Horizontal" H 1800 1700 50  0001 C CNN
+F 2 "BBS Components:USB_B_Male_Molex_0480370001" H 1800 1700 50  0001 C CNN
 F 3 " ~" H 1800 1700 50  0001 C CNN
 	1    1650 1750
@@
 F 0 "J2" H 2670 1739 50  0000 R CNN
 F 1 "USB_A" H 2670 1648 50  0000 R CNN
-F 2 "Connector_USB:USB_A_Stewart_SS-52100-001_Horizontal" H 3050 1700 50  0001 C CNN
+F 2 "BBS Components:USB_A_Female_Molex_0676432910" H 3050 1700 50  0001 C CNN
 F 3 " ~" H 3050 1700 50  0001 C CNN
 	1    2900 1750
@@
 F 0 "R1" H 2320 2146 50  0000 L CNN
 F 1 "R" H 2320 2055 50  0000 L CNN
-F 2 "Resistor_SMD:R_0603_1608Metric_Pad1.05x0.95mm_HandSolder" V 2180 2100 50  0001 C CNN
+F 2 "BBS Components:R_0603_HandSoldering_NoSilk" V 2180 2100 50  0001 C CNN
 F 3 "~" H 2250 2100 50  0001 C CNN
 	1    2250 2100
@@
 F 0 "D1" V 2289 2433 50  0000 R CNN
 F 1 "LED" V 2198 2433 50  0000 R CNN
-F 2 "LED_SMD:LED_0603_1608Metric_Pad1.05x0.95mm_HandSolder" H 2250 2550 50  0001 C CNN
+F 2 "BBS Components:LED_0603_HandSoldering" H 2250 2550 50  0001 C CNN
 F 3 "~" H 2250 2550 50  0001 C CNN
 	1    2250 2550
